File: Eagle/controldeveloper/Main.brd (EAGLE design)
At the start: 60 x 65 mm, 19 parts

Commit message: Added encoders on Eagle Project
Parts:
- added JP1, JP2: (no value), pinhead:1X03/90
Connections:
- new net N$17: JP1.3
- new net N$18: JP2.3
- net GND: now also JP1.1, JP2.1
- net VCC: now also JP1.2, JP2.2
Changed lines of the file:
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@@
 <setting verticaltext="up"/>
 </settings>
-<grid distance="1" unitdist="mm" unit="mm" style="lines" multiple="1" display="yes" altdistance="0.1" altunitdist="mm" altunit="mm"/>
+<grid distance="1" unitdist="mm" unit="mm" style="lines" multiple="1" display="yes" altdistance="0.5" altunitdist="mm" altunit="mm"/>
 <layers>
 <layer number="1" name="Top" color="4" fill="1" visible="yes" active="yes"/>
@@
 <element name="U3" library="MicroUSB" package="USB-MICRO-SMD" value="" x="18" y="3" rot="R90"/>
 <element name="ESP_L" library="pinhead" package="2X09" value="" x="29.5" y="23.6"/>
+<element name="JP1" library="pinhead" package="1X03/90" value="" x="-7" y="6"/>
+<element name="JP2" library="pinhead" package="1X03/90" value="" x="-20" y="6"/>
 </elements>
 <signals>
@@
 <wire x1="46" y1="16" x2="44" y2="14" width="1.27" layer="1"/>
 <wire x1="44" y1="14" x2="22.9" y2="14" width="1.27" layer="1"/>
+<contactref element="JP1" pad="1"/>
+<contactref element="JP2" pad="1"/>
 <wire x1="13.57" y1="52.43" x2="12" y2="37.54" width="0" layer="19" extent="16-16"/>
+<wire x1="-9.54" y1="2.19" x2="19.3" y2="5.7" width="0" layer="19" extent="1-1"/>
+<wire x1="-22.54" y1="2.19" x2="-9.54" y2="2.19" width="0" layer="19" extent="1-1"/>
 </signal>
 <signal name="N$1">
@@
 <via x="48" y="14" extent="1-16" drill="0.6" shape="square"/>
 <wire x1="48" y1="14" x2="28" y2="14" width="1.27" layer="16"/>
+<contactref element="JP1" pad="2"/>
+<contactref element="JP2" pad="2"/>
+<wire x1="-7" y1="2.19" x2="13" y2="15" width="0" layer="19" extent="16-16"/>
+<wire x1="-20" y1="2.19" x2="-7" y2="2.19" width="0" layer="19" extent="1-1"/>
+</signal>
+<signal name="N$17">
+<contactref element="JP1" pad="3"/>
+</signal>
+<signal name="N$18">
+<contactref element="JP2" pad="3"/>
 </signal>
 </signals>

Commit message: Eagle proj - redesigned
Parts:
- removed JP1, JP2: (no value), pinhead:1X03/90
- added ENC_R, EN_L: (no value), pinhead:1X03
- moved C5 50.8 mm to (4.41, 6.29), turned to 0 degrees
- moved C4 43.7 mm to (51.1, 15.4), turned to 0 degrees
- moved M_OUT 24.9 mm to (58.0, 9.05), turned to 270 degrees
- moved R5 20.1 mm to (40.9, 51.2), turned to 90 degrees
- moved C6 14.4 mm to (3.98, 14.3)
- moved LED1 13.6 mm to (33.5, 60.4)
- moved C7 10.3 mm to (50.5, 21.3), turned to 0 degrees
- moved IN 9.02 mm to (40.1, 10.6)
- moved OUT 8.23 mm to (40.1, 3.64)
- moved R2 8.13 mm to (46.2, 32.1), turned to 0 degrees
- moved RX/TX 6.95 mm to (24.0, 58.0)
- moved R4 6.11 mm to (44.9, 51.0)
- moved ESP_R 5.41 mm to (24.6, 51.4)
- moved ESP_L 4.59 mm to (32.1, 19.8)
- moved R1 4.40 mm to (14.1, 45.9)
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Connections:
- net N$11 renamed VDD
- removed net N$17: JP1.3
- removed net N$18: JP2.3
- removed net N$5: ESP_R.4, RX/TX.1
- removed net N$8: ESP_R.3, R1.1
- new net EN1: ESP_L.8, IN.3
- new net EN2: ESP_L.10, IN.5
- new net ENC_L: EN_L.3, ESP_L.4
- new net ENC_R: ENC_R.3, ESP_R.18
- new net LED1: ESP_R.9, R5.1
- new net LED2: ESP_R.11, R4.1
- new net N$12: ESP_R.5, R1.1
- new net N$14: ESP_R.8, RX/TX.2
- new net PH1: ESP_L.9, IN.4
- new net PH2: ESP_L.7, IN.6
- net GND: now also ENC_R.1, EN_L.1, ESP_R.3; no longer ESP_R.1, JP1.1, JP2.1
- net N$6: now also RX/TX.1; no longer RX/TX.2
- net N$9: now also ESP_R.10; no longer ESP_R.8
- net VCC: now also ENC_R.2, EN_L.2, ESP_R.4; no longer ESP_R.2, JP1.2, JP2.2
Routing:
- net GND: track 166.3 -> 0.00 mm, vias 5 -> 0
- net VCC: track 117.0 -> 0.00 mm, vias 2 -> 0
- net VDD: track 86.5 -> 0.00 mm, vias 1 -> 0
- net N$13: track 22.5 -> 0.00 mm
- net N$7: track 17.2 -> 0.00 mm
- net N$5: track 9.48 -> 0.00 mm
- net N$9: track 9.42 -> 0.00 mm
- net N$6: track 9.42 -> 0.00 mm
- net N$8: track 8.93 -> 0.00 mm
- net N$4: track 7.25 -> 0.00 mm
- net N$3: track 7.25 -> 0.00 mm
- net N$2: track 7.25 -> 0.00 mm
- net N$1: track 7.25 -> 0.00 mm
- net N$10: track 4.76 -> 0.00 mm
Other:
- board size 60 x 65 mm -> 64 x 81 mm

Commit message: Finished eagle board!
Parts:
- removed IC2: (no value), v-reg:317TL
- added IC1: (no value), v-reg:317TS
- moved EN_L 56.8 mm to (8.01, 51.8)
- moved ENC_R 55.2 mm to (52.0, 51.9)
- moved C5 47.3 mm to (51.7, 6.41), turned to 90 degrees
- moved M_OUT 36.9 mm to (21.4, 3.99), turned to 0 degrees
- moved C6 36.1 mm to (40.0, 11.3)
- moved RX/TX 32.5 mm to (52.0, 41.5), turned to 270 degrees
- moved C7 32.0 mm to (44.5, 52.7), turned to 180 degrees
- moved U3 27.0 mm to (40.9, 4.06)
- moved C4 26.9 mm to (28.9, 30.6), turned to 180 degrees
- moved ESP_R 24.8 mm to (44.4, 36.4), turned to 270 degrees
- moved ESP_L 24.3 mm to (14.3, 36.4), turned to 270 degrees
- moved IN 21.5 mm to (20.1, 18.6)
- moved OUT 21.2 mm to (20.1, 10.6)
- moved R3 19.3 mm to (28.6, 34.1)
- moved R5 18.9 mm to (22.8, 56.9), turned to 180 degrees
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Connections:
- removed net N$14: ESP_R.8, RX/TX.2
- removed net N$9: ESP_R.10, RX/TX.3
- new net N$5: ESP_R.4, RX/TX.1
- new net N$8: ESP_R.8, RX/TX.3
- net ENC_R: now also ESP_R.16; no longer ESP_R.18
- net GND: now also ESP_R.1; no longer ESP_R.3
- net LED1: now also ESP_R.7; no longer ESP_R.9
- net LED2: now also ESP_R.9; no longer ESP_R.11
- net N$12: now also ESP_R.3; no longer ESP_R.5
- net N$6: now also RX/TX.2; no longer RX/TX.1
- net N$7: now also IC1.1; no longer IC2.1
- net VCC: now also ESP_R.2, IC1.2; no longer ESP_R.4, IC2.2
- net VDD: now also IC1.3; no longer IC2.3
Routing:
- net GND: track 0.00 -> 254.5 mm, vias 0 -> 5
- net VCC: track 0.00 -> 193.7 mm, vias 0 -> 2
- net VDD: track 0.00 -> 100.7 mm, vias 0 -> 1
- net PH2: track 0.00 -> 57.1 mm, vias 0 -> 2
- net ENC_R: track 0.00 -> 37.3 mm
- net PH1: track 0.00 -> 36.2 mm, vias 0 -> 2
- net ENC_L: track 0.00 -> 32.5 mm
- net EN2: track 0.00 -> 31.8 mm, vias 0 -> 2
- net EN1: track 0.00 -> 29.0 mm
- net LED1: track 0.00 -> 26.0 mm
- net N$7: track 0.00 -> 26.0 mm
- net LED2: track 0.00 -> 23.7 mm, vias 0 -> 2
- net N$12: track 0.00 -> 13.5 mm
- net N$13: track 0.00 -> 7.90 mm
- net N$10: track 0.00 -> 6.93 mm
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Other:
- board size 64 x 81 mm -> 60 x 65 mm
